File: mysensors/node/livolo_EU_switch/VL-C700X-1_Ver_C2/NRF51822/1_channel/livolo_1_channel_1way_eu_switch.kicad_pcb (KiCad board)
At the start: 2 copper layers, 43 x 43.4 mm, 31 parts, among them J1 SWD, P4 Power Board, U1 Touch, U2 MCP16301, U3 MTCH102, U5 PTR5518

Commit message: livolo nrf51822 refactorings
Parts:
- added J2: 3V_EN, Connectors:GS2, B.Cu at (146.6, 108.7)
Connections:
- P4 pad 1: Net-(P4-Pad1) -> (no net)
- P4 pad 10: Net-(P4-Pad10) -> (no net)
- P4 pad 12: Net-(P4-Pad12) -> (no net)
- P4 pad 14: Net-(P4-Pad14) -> (no net)
- P4 pad 7: Net-(P4-Pad7) -> (no net)
- P4 pad 8: Net-(P4-Pad8) -> (no net)
- P4 pad 9: Net-(P4-Pad9) -> (no net)
- U5 pad 6: (no net) -> Net-(U5-Pad6)
- U5 pad 7: Net-(U5-Pad7) -> (no net)
- U5 pad 8: Net-(U5-Pad8) -> (no net)
Routing:
- net +3V3: track 66.5 -> 72.5 mm
- net Net-(J2-Pad1): track 0.00 -> 3.04 mm
Other:
- board text added: "Rev. 0.3"
- board text removed: "Rev. 0.2"
Changed lines of the file:
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@@
-(kicad_pcb (version 20170123) (host pcbnew no-vcs-found-3ac87f6~59~ubuntu16.04.1)
+(kicad_pcb (version 20170922) (host pcbnew no-vcs-found-6573a43~60~ubuntu16.04.1)
   (general
     (thickness 1.6)
     (drawings 37)
-    (tracks 228)
+    (tracks 232)
     (zones 0)
-    (modules 31)
-    (nets 35)
+    (modules 32)
+    (nets 27)
   )
   (page A4)
@@
   (net 23 /MTSA)
   (net 24 /MTPM)
-  (net 25 "Net-(P4-Pad14)")
-  (net 26 "Net-(P4-Pad13)")
-  (net 27 "Net-(P4-Pad12)")
-  (net 28 "Net-(P4-Pad10)")
-  (net 29 "Net-(P4-Pad9)")
-  (net 30 "Net-(P4-Pad8)")
-  (net 31 "Net-(P4-Pad7)")
-  (net 32 "Net-(P4-Pad1)")
-  (net 33 "Net-(U5-Pad8)")
-  (net 34 "Net-(U5-Pad7)")
+  (net 25 "Net-(J2-Pad1)")
+  (net 26 "Net-(U5-Pad6)")
   (net_class Default "This is the default net class."
     (clearance 0.25)
@@
     (add_net "Net-(D5-Pad1)")
     (add_net "Net-(D6-Pad2)")
-    (add_net "Net-(P4-Pad1)")
-    (add_net "Net-(P4-Pad10)")
-    (add_net "Net-(P4-Pad12)")
-    (add_net "Net-(P4-Pad13)")
-    (add_net "Net-(P4-Pad14)")
-    (add_net "Net-(P4-Pad7)")
-    (add_net "Net-(P4-Pad8)")
-    (add_net "Net-(P4-Pad9)")
+    (add_net "Net-(J2-Pad1)")
     (add_net "Net-(R1-Pad1)")
     (add_net "Net-(R3-Pad1)")
@@
     (add_net "Net-(R4-Pad1)")
     (add_net "Net-(R4-Pad2)")
-    (add_net "Net-(U5-Pad7)")
-    (add_net "Net-(U5-Pad8)")
+    (add_net "Net-(U5-Pad6)")
   )
   (module w_logo:Logo_silk_OSHW_6x6mm locked (layer B.Cu)
@@
     (pad 10 smd rect (at -8.1294 -1.4732 270) (size 0.8128 2.5) (layers F.Cu F.Paste F.Mask)
       (net 1 +3V3))
-    (pad 6 smd rect (at 7.3166 -1.4732 270) (size 0.8128 2.5) (layers F.Cu F.Paste F.Mask))
+    (pad 6 smd rect (at 7.3166 -1.4732 270) (size 0.8128 2.5) (layers F.Cu F.Paste F.Mask)
+      (net 26 "Net-(U5-Pad6)"))
     (pad 9 smd rect (at -8.1294 -2.7432 270) (size 0.8128 2.5) (layers F.Cu F.Paste F.Mask)
       (net 2 GND))
-    (pad 7 smd rect (at 7.3166 -2.7432 270) (size 0.8128 2.5) (layers F.Cu F.Paste F.Mask)
-      (net 34 "Net-(U5-Pad7)"))
-    (pad 8 smd rect (at 7.3166 -4.0132 270) (size 0.8128 2.5) (layers F.Cu F.Paste F.Mask)
-      (net 33 "Net-(U5-Pad8)"))
+    (pad 7 smd rect (at 7.3166 -2.7432 270) (size 0.8128 2.5) (layers F.Cu F.Paste F.Mask))
+    (pad 8 smd rect (at 7.3166 -4.0132 270) (size 0.8128 2.5) (layers F.Cu F.Paste F.Mask))
     (model ${KISYS3DMOD}/Radio_Modules.3dshapes/PTR5518.stp
       (at (xyz 0 0 0))
@@
     (fp_line (start -1 13) (end 3 13) (layer F.Fab) (width 0.1))
     (fp_line (start -1 -1) (end -1 13) (layer F.Fab) (width 0.1))
-    (pad 14 thru_hole oval (at 2 12 90) (size 1.35 1.35) (drill 0.8) (layers *.Cu *.Mask)
-      (net 25 "Net-(P4-Pad14)"))
+    (pad 14 thru_hole oval (at 2 12 90) (size 1.35 1.35) (drill 0.8) (layers *.Cu *.Mask))
     (pad 13 thru_hole oval (at 0 12 90) (size 1.35 1.35) (drill 0.8) (layers *.Cu *.Mask)
-      (net 26 "Net-(P4-Pad13)"))
-    (pad 12 thru_hole oval (at 2 10 90) (size 1.35 1.35) (drill 0.8) (layers *.Cu *.Mask)
-      (net 27 "Net-(P4-Pad12)"))
+      (net 25 "Net-(J2-Pad1)"))
+    (pad 12 thru_hole oval (at 2 10 90) (size 1.35 1.35) (drill 0.8) (layers *.Cu *.Mask))
     (pad 11 thru_hole oval (at 0 10 90) (size 1.35 1.35) (drill 0.8) (layers *.Cu *.Mask)
       (net 2 GND))
-    (pad 10 thru_hole oval (at 2 8 90) (size 1.35 1.35) (drill 0.8) (layers *.Cu *.Mask)
-      (net 28 "Net-(P4-Pad10)"))
-    (pad 9 thru_hole oval (at 0 8 90) (size 1.35 1.35) (drill 0.8) (layers *.Cu *.Mask)
-      (net 29 "Net-(P4-Pad9)"))
-    (pad 8 thru_hole oval (at 2 6 90) (size 1.35 1.35) (drill 0.8) (layers *.Cu *.Mask)
-      (net 30 "Net-(P4-Pad8)"))
-    (pad 7 thru_hole oval (at 0 6 90) (size 1.35 1.35) (drill 0.8) (layers *.Cu *.Mask)
-      (net 31 "Net-(P4-Pad7)"))
+    (pad 10 thru_hole oval (at 2 8 90) (size 1.35 1.35) (drill 0.8) (layers *.Cu *.Mask))
+    (pad 9 thru_hole oval (at 0 8 90) (size 1.35 1.35) (drill 0.8) (layers *.Cu *.Mask))
+    (pad 8 thru_hole oval (at 2 6 90) (size 1.35 1.35) (drill 0.8) (layers *.Cu *.Mask))
+    (pad 7 thru_hole oval (at 0 6 90) (size 1.35 1.35) (drill 0.8) (layers *.Cu *.Mask))
     (pad 6 thru_hole oval (at 2 4 90) (size 1.35 1.35) (drill 0.8) (layers *.Cu *.Mask)
       (net 13 /Relay1_Reset))
@@
     (pad 2 thru_hole oval (at 2 0 90) (size 1.35 1.35) (drill 0.8) (layers *.Cu *.Mask)
       (net 6 /12Vcc))
-    (pad 1 thru_hole rect (at 0 0 90) (size 1.35 1.35) (drill 0.8) (layers *.Cu *.Mask)
-      (net 32 "Net-(P4-Pad1)"))
+    (pad 1 thru_hole rect (at 0 0 90) (size 1.35 1.35) (drill 0.8) (layers *.Cu *.Mask))
     (model ${KISYS3DMOD}/Pin_Headers.3dshapes/Female/female_header_2row_14pins_2mm.step
       (at (xyz 0 0 0))
@@
       (net 20 "Net-(R3-Pad2)"))
   )
+  (module Connectors:GS2 (layer B.Cu)
+    (at 146.6 108.7)
+    (descr "2-pin solder bridge")
+    (tags "solder bridge")
+    (attr smd)
+    (fp_text reference J2 (at 0.5 -2.2 -90) (layer B.SilkS)
+      (effects (font (size 0.5 0.5) (thickness 0.1)) (justify mirror))
+    )
+    (fp_text value 3V_EN (at -0.5 -2.7 -90) (layer B.SilkS)
+      (effects (font (size 0.5 0.5) (thickness 0.1)) (justify mirror))
+    )
+    (fp_line (start -0.89 1.27) (end 0.89 1.27) (layer B.SilkS) (width 0.12))
+    (fp_line (start 0.89 -1.27) (end -0.89 -1.27) (layer B.SilkS) (width 0.12))
+    (fp_line (start 0.89 -1.27) (end 0.89 1.27) (layer B.SilkS) (width 0.12))
+    (fp_line (start -0.89 1.27) (end -0.89 -1.27) (layer B.SilkS) (width 0.12))
+    (fp_line (start -1.1 1.45) (end 1.1 1.45) (layer B.CrtYd) (width 0.05))
+    (fp_line (start -1.1 -1.5) (end -1.1 1.45) (layer B.CrtYd) (width 0.05))
+    (fp_line (start 1.1 -1.5) (end -1.1 -1.5) (layer B.CrtYd) (width 0.05))
+    (fp_line (start 1.1 1.45) (end 1.1 -1.5) (layer B.CrtYd) (width 0.05))
+    (pad 2 smd rect (at 0 -0.64) (size 1.27 0.97) (layers B.Cu B.Paste B.Mask)
+      (net 1 +3V3))
+    (pad 1 smd rect (at 0 0.64) (size 1.27 0.97) (layers B.Cu B.Paste B.Mask)
+      (net 25 "Net-(J2-Pad1)"))
+  )
   (gr_line (start 134.4 75.30098) (end 150 75.30098) (layer Edge.Cuts) (width 0.1))
   (gr_line (start 150 75.30098) (end 150 70.2) (layer Edge.Cuts) (width 0.1))
@@
     (effects (font (size 0.6 0.6) (thickness 0.12)) (justify mirror))
   )
-  (gr_text "Rev. 0.2" (at 125.6 106.3 90) (layer F.SilkS)
+  (gr_text "Rev. 0.3" (at 125.6 106.3 90) (layer F.SilkS)
     (effects (font (size 1 1) (thickness 0.2)))
   )
@@
     (effects (font (size 1.2 1.2) (thickness 0.2)) (justify mirror))
   )
+  (segment (start 145.1 102.05) (end 146.6 102.05) (width 0.3) (layer B.Cu) (net 1) (status 10))
+  (segment (start 146.6 102.05) (end 149.75 102.05) (width 0.3) (layer B.Cu) (net 1))
+  (segment (start 146.6 108.06) (end 146.6 102.05) (width 0.3) (layer B.Cu) (net 1) (status 10))
   (segment (start 156.999996 88.6) (end 156.999996 88.599996) (width 0.3) (layer B.Cu) (net 1))
   (segment (start 156.999996 88.599996) (end 156.6 88.2) (width 0.3) (layer B.Cu) (net 1))
@@
   (segment (start 157.1 89.8) (end 157.1 88.700004) (width 0.3) (layer F.Cu) (net 1) (status 10))
   (via (at 156.999996 88.6) (size 0.8) (drill 0.4) (layers F.Cu B.Cu) (net 1))
-  (segment (start 145.1 102.05) (end 149.75 102.05) (width 0.3) (layer B.Cu) (net 1) (status 10))
   (segment (start 149.75 102.05) (end 151.2 100.6) (width 0.3) (layer B.Cu) (net 1))
   (via (at 151.2 100.6) (size 0.8) (drill 0.4) (layers F.Cu B.Cu) (net 1))
@@
   (segment (start 155.6 93.575) (end 155.6 95) (width 0.3) (layer F.Cu) (net 24) (status 10))
   (via (at 155.6 95) (size 0.8) (drill 0.4) (layers F.Cu B.Cu) (net 24))
+  (segment (start 143.65 109.55) (end 146.39 109.55) (width 0.3) (layer B.Cu) (net 25) (status 30))
+  (segment (start 146.39 109.55) (end 146.6 109.34) (width 0.25) (layer B.Cu) (net 25) (status 30))
   (zone (net 2) (net_name GND) (layer F.Cu) (hatch edge 0.508)
     (connect_pads (clearance 0.45))

Commit message: livolo nrf51822 boards refactorings, opi zero
Parts:
- removed G***: LOGO, w_logo:Logo_silk_OSHW_6x6mm
- added REF***: KiCad-Logo2_6mm_SilkScreen, Symbols:KiCad-Logo2_6mm_SilkScreen, F.Cu at (159.0, 91.8)
- moved R8 37.6 mm to (125.2, 86.5), turned to 180 degrees
- moved C4 35.4 mm to (125.2, 88.1), turned to 0 degrees
- moved R7 31.6 mm to (126.8, 93.7), turned to 0 degrees
- moved U3 30.6 mm to (127.2, 90.9), turned to 180 degrees
- moved C3 26.5 mm to (129.6, 94.7), turned to 90 degrees
- moved R3 21.2 mm to (132.2, 89.5), turned to 0 degrees
- moved R4 20.6 mm to (132.2, 91.3), turned to 0 degrees
- moved C7 2.20 mm to (153.0, 102.5), turned to 180 degrees
- moved C1 1.25 mm to (131.6, 79.3), turned to 90 degrees
- moved C2 1.25 mm to (129.5, 79.3), turned to 270 degrees
- moved U1 0.51 mm to (142.3, 92.3), turned to 225 degrees
Connections:
- J1 pad 2: +3V3 -> GND
- J1 pad 4: GND -> +3V3
- P4 pad 1: (no net) -> Net-(P4-Pad1)
- P4 pad 10: (no net) -> Net-(P4-Pad10)
- P4 pad 12: (no net) -> Net-(P4-Pad12)
- P4 pad 14: (no net) -> Net-(P4-Pad14)
- P4 pad 7: (no net) -> Net-(P4-Pad7)
- P4 pad 8: (no net) -> Net-(P4-Pad8)
- P4 pad 9: (no net) -> Net-(P4-Pad9)
- U5 pad 1: /TS1 -> /S1_LEDs
- U5 pad 11: /S1_LEDs -> Net-(U5-Pad11)
- U5 pad 13: /Relay1_Reset -> /MTSA
- U5 pad 14: /Relay2_Set -> /TS1
- U5 pad 15: /Relay2_Reset -> /MTPM
- U5 pad 2: /MTSA -> Net-(U5-Pad2)
- U5 pad 3: /MTPM -> Net-(U5-Pad3)
- U5 pad 6: Net-(U5-Pad6) -> /Relay2_Set
- U5 pad 7: (no net) -> /Relay1_Reset
- U5 pad 8: (no net) -> /Relay2_Reset
Routing:
- net GND: track 73.9 -> 47.4 mm
- net /S1_LEDs: track 44.6 -> 29.6 mm, vias 2 -> 0
- net /Relay2_Reset: track 35.3 -> 49.0 mm, vias 0 -> 1
- net +3V3: track 72.5 -> 85.8 mm
- net /Relay1_Reset: track 33.3 -> 45.6 mm, vias 2 -> 1
- net /MTPM: track 17.4 -> 7.82 mm, vias 2 -> 0
- net /Relay2_Set: track 40.0 -> 47.5 mm, vias 0 -> 1
- net /MTSA: track 16.3 -> 9.94 mm
- net /TS1: track 15.9 -> 17.3 mm
- net Net-(C4-Pad1): track 5.03 -> 3.78 mm
- net Net-(R3-Pad2): track 13.8 -> 14.5 mm
- net /Relay1_Set: track 34.1 -> 34.0 mm, vias 2 -> 1
Other:
- board text removed: "Mysensors NRF51822 Livolo Node"
