File: mysensors/node/livolo_EU_switch/VL-C700X-1_Ver_C2/NRF51822/2_channel/livolo_2_channels_1way_eu_switch.kicad_pcb (KiCad board)
At the start: 2 copper layers, 43.5 x 43.4 mm, 42 parts, among them J1 SWD, J2 3V_EN, P4 Power Board, U1 Touch, U2 MCP16301, U5 PTR5518, U6 Touch, U7 MTCH105

Commit message: livolo nrf51822 boards refactorings, opi zero
Parts:
- removed G***: LOGO, w_logo:Logo_silk_OSHW_6x6mm
- added REF***: KiCad-Logo2_6mm_SilkScreen, Symbols:KiCad-Logo2_6mm_SilkScreen, F.Cu at (124.5, 84.5)
Other:
- board text removed: "Mysensors NRF51822 Livolo Node"
