File: esp8266_shields/uno_relay/esp8266_uno_relay.kicad_pcb (KiCad board)
At the start: 2 copper layers, 68.8 x 53.2 mm, 221 parts, among them J1 GS2, J10 R_CON, J2 GS2, J3 GS2, J4 GS2, J5 GS2, J6 GS2, J7 GS2, J8 GS2, J9 GS2, K1 SLA-05VDC-SL-C, Q1 MMBT2222, SW1 RESET

Commit message: esp8266 uno relay shield refactorings
Parts:
- removed the REF*** at (116.8, 123.8)
- removed V10_10, V10_11, V10_12, V10_13, V10_14, V10_16, V10_17, V10_18, V10_21, V10_4, V10_5, V10_6, V10_7, V10_8, V10_9, V11_17, V11_18, V11_4, V11_5, V11_6, V11_7, V12_16, V12_18, V12_4, V12_5, V12_6, V12_7, V13_16, V13_17, V13_4, V13_5, V13_6, V13_7, V14_18, V14_4, V14_5, V15_4, V15_5, V16_20, V16_4, V16_5, V17_19, V17_4, V17_5, V18_19, V18_20, V18_4, V19_20, V19_5, V20_2, V20_5, V22_21, V4_10, V4_11, V4_12, V4_13, V4_14, V4_15, V4_16, V4_17, V4_18, V4_19, V4_20, V4_21, V4_5, V4_6, V4_7, V4_8, V4_9, V5_10, V5_11, V5_12, V5_13, V5_14, V5_15, V5_16, V5_17, V5_18, V5_19, V5_20, V5_21, V5_4, V5_5, V5_6, V5_7, V5_8, V5_9, V6_12, V6_13, V6_14, V6_15, V6_16, V6_17, V6_18, V7_10, V7_11, V7_13, V7_14, V7_15, V7_16, V7_17, V7_18, V7_21, V7_5, V7_6, V7_7, V7_8, V7_9, V8_10, V8_11, V8_12, V8_14, V8_15, V8_16, V8_17, V8_18, V8_19, V8_20, V8_4, V8_5, V8_6, V8_7, V8_8, V8_9, V9_10, V9_11, V9_12, V9_13, V9_15, V9_16, V9_17, V9_18, V9_4, V9_5, V9_6, V9_7, V9_8, V9_9: AUTO_VIA, VIA_MATRIX
- added REF**: SolderWirePad_single_0-8mmDrill, Wire_Pads:SolderWirePad_single_0-8mmDrill, F.Cu at (133.3, 102.3)
- added REF**: SolderWirePad_single_0-8mmDrill, Wire_Pads:SolderWirePad_single_0-8mmDrill, F.Cu at (125.6, 110.0)
- added REF**: SolderWirePad_single_0-8mmDrill, Wire_Pads:SolderWirePad_single_0-8mmDrill, F.Cu at (107.8, 112.5)
- added REF**: SolderWirePad_single_0-8mmDrill, Wire_Pads:SolderWirePad_single_0-8mmDrill, F.Cu at (120.5, 109.9)
- added REF**: SolderWirePad_single_0-8mmDrill, Wire_Pads:SolderWirePad_single_0-8mmDrill, F.Cu at (117.9, 109.9)
- added REF**: SolderWirePad_single_0-8mmDrill, Wire_Pads:SolderWirePad_single_0-8mmDrill, F.Cu at (115.4, 109.9)
- added REF**: SolderWirePad_single_0-8mmDrill, Wire_Pads:SolderWirePad_single_0-8mmDrill, F.Cu at (112.8, 109.9)
- added REF**: SolderWirePad_single_0-8mmDrill, Wire_Pads:SolderWirePad_single_0-8mmDrill, F.Cu at (110.3, 109.9)
- added REF**: SolderWirePad_single_0-8mmDrill, Wire_Pads:SolderWirePad_single_0-8mmDrill, F.Cu at (107.8, 109.9)
- added REF**: SolderWirePad_single_0-8mmDrill, Wire_Pads:SolderWirePad_single_0-8mmDrill, F.Cu at (120.5, 107.4)
- added REF**: SolderWirePad_single_0-8mmDrill, Wire_Pads:SolderWirePad_single_0-8mmDrill, F.Cu at (117.9, 107.4)
- added REF**: SolderWirePad_single_0-8mmDrill, Wire_Pads:SolderWirePad_single_0-8mmDrill, F.Cu at (115.4, 107.4)
- added REF**: SolderWirePad_single_0-8mmDrill, Wire_Pads:SolderWirePad_single_0-8mmDrill, F.Cu at (123.1, 130.3)
- added REF**: SolderWirePad_single_0-8mmDrill, Wire_Pads:SolderWirePad_single_0-8mmDrill, F.Cu at (112.8, 107.4)
- added REF**: SolderWirePad_single_0-8mmDrill, Wire_Pads:SolderWirePad_single_0-8mmDrill, F.Cu at (110.3, 107.4)
- added REF**: SolderWirePad_single_0-8mmDrill, Wire_Pads:SolderWirePad_single_0-8mmDrill, F.Cu at (107.8, 107.4)
- added REF**: SolderWirePad_single_0-8mmDrill, Wire_Pads:SolderWirePad_single_0-8mmDrill, F.Cu at (120.5, 104.8)
- added REF**: SolderWirePad_single_0-8mmDrill, Wire_Pads:SolderWirePad_single_0-8mmDrill, F.Cu at (117.9, 104.8)
- added REF**: SolderWirePad_single_0-8mmDrill, Wire_Pads:SolderWirePad_single_0-8mmDrill, F.Cu at (115.4, 104.8)
- added REF**: SolderWirePad_single_0-8mmDrill, Wire_Pads:SolderWirePad_single_0-8mmDrill, F.Cu at (112.8, 104.8)
- added REF**: SolderWirePad_single_0-8mmDrill, Wire_Pads:SolderWirePad_single_0-8mmDrill, F.Cu at (110.3, 104.8)
- added REF**: SolderWirePad_single_0-8mmDrill, Wire_Pads:SolderWirePad_single_0-8mmDrill, F.Cu at (107.8, 104.8)
- added REF**: SolderWirePad_single_0-8mmDrill, Wire_Pads:SolderWirePad_single_0-8mmDrill, F.Cu at (120.5, 102.3)
- added REF**: SolderWirePad_single_0-8mmDrill, Wire_Pads:SolderWirePad_single_0-8mmDrill, F.Cu at (130.7, 132.8)
- added REF**: SolderWirePad_single_0-8mmDrill, Wire_Pads:SolderWirePad_single_0-8mmDrill, F.Cu at (117.9, 102.3)
- added REF**: SolderWirePad_single_0-8mmDrill, Wire_Pads:SolderWirePad_single_0-8mmDrill, F.Cu at (115.4, 102.3)
- added REF**: SolderWirePad_single_0-8mmDrill, Wire_Pads:SolderWirePad_single_0-8mmDrill, F.Cu at (112.8, 102.3)
- added REF**: SolderWirePad_single_0-8mmDrill, Wire_Pads:SolderWirePad_single_0-8mmDrill, F.Cu at (110.3, 102.3)
- added REF**: SolderWirePad_single_0-8mmDrill, Wire_Pads:SolderWirePad_single_0-8mmDrill, F.Cu at (107.8, 102.3)
- added REF**: SolderWirePad_single_0-8mmDrill, Wire_Pads:SolderWirePad_single_0-8mmDrill, F.Cu at (120.5, 99.8)
- added REF**: SolderWirePad_single_0-8mmDrill, Wire_Pads:SolderWirePad_single_0-8mmDrill, F.Cu at (117.9, 99.8)
- added REF**: SolderWirePad_single_0-8mmDrill, Wire_Pads:SolderWirePad_single_0-8mmDrill, F.Cu at (115.4, 99.8)
- added REF**: SolderWirePad_single_0-8mmDrill, Wire_Pads:SolderWirePad_single_0-8mmDrill, F.Cu at (112.8, 99.8)
- added REF**: SolderWirePad_single_0-8mmDrill, Wire_Pads:SolderWirePad_single_0-8mmDrill, F.Cu at (110.3, 99.8)
- added REF**: SolderWirePad_single_0-8mmDrill, Wire_Pads:SolderWirePad_single_0-8mmDrill, F.Cu at (128.2, 130.3)
- added REF**: SolderWirePad_single_0-8mmDrill, Wire_Pads:SolderWirePad_single_0-8mmDrill, F.Cu at (107.8, 99.8)
- added REF**: SolderWirePad_single_0-8mmDrill, Wire_Pads:SolderWirePad_single_0-8mmDrill, F.Cu at (128.2, 135.3)
- added REF**: SolderWirePad_single_0-8mmDrill, Wire_Pads:SolderWirePad_single_0-8mmDrill, F.Cu at (128.2, 132.8)
- added REF**: SolderWirePad_single_0-8mmDrill, Wire_Pads:SolderWirePad_single_0-8mmDrill, F.Cu at (125.6, 127.8)
- added REF**: SolderWirePad_single_0-8mmDrill, Wire_Pads:SolderWirePad_single_0-8mmDrill, F.Cu at (130.7, 135.3)
- added REF**: SolderWirePad_single_0-8mmDrill, Wire_Pads:SolderWirePad_single_0-8mmDrill, F.Cu at (125.6, 135.3)
- added REF**: SolderWirePad_single_0-8mmDrill, Wire_Pads:SolderWirePad_single_0-8mmDrill, F.Cu at (130.7, 130.3)
- added REF**: SolderWirePad_single_0-8mmDrill, Wire_Pads:SolderWirePad_single_0-8mmDrill, F.Cu at (138.4, 99.8)
- added REF**: SolderWirePad_single_0-8mmDrill, Wire_Pads:SolderWirePad_single_0-8mmDrill, F.Cu at (125.6, 132.8)
- added REF**: SolderWirePad_single_0-8mmDrill, Wire_Pads:SolderWirePad_single_0-8mmDrill, F.Cu at (123.1, 127.8)
- added REF**: SolderWirePad_single_0-8mmDrill, Wire_Pads:SolderWirePad_single_0-8mmDrill, F.Cu at (125.6, 130.3)
- added REF**: SolderWirePad_single_0-8mmDrill, Wire_Pads:SolderWirePad_single_0-8mmDrill, F.Cu at (123.1, 132.8)
- added REF**: SolderWirePad_single_0-8mmDrill, Wire_Pads:SolderWirePad_single_0-8mmDrill, F.Cu at (123.1, 135.3)
- added REF**: SolderWirePad_single_0-8mmDrill, Wire_Pads:SolderWirePad_single_0-8mmDrill, F.Cu at (130.7, 107.3)
- added REF**: SolderWirePad_single_0-8mmDrill, Wire_Pads:SolderWirePad_single_0-8mmDrill, F.Cu at (128.2, 107.3)
- added REF**: SolderWirePad_single_0-8mmDrill, Wire_Pads:SolderWirePad_single_0-8mmDrill, F.Cu at (125.6, 107.3)
- added REF**: SolderWirePad_single_0-8mmDrill, Wire_Pads:SolderWirePad_single_0-8mmDrill, F.Cu at (123.1, 107.3)
- added REF**: SolderWirePad_single_0-8mmDrill, Wire_Pads:SolderWirePad_single_0-8mmDrill, F.Cu at (125.6, 104.8)
- added REF**: SolderWirePad_single_0-8mmDrill, Wire_Pads:SolderWirePad_single_0-8mmDrill, F.Cu at (140.9, 99.8)
- added REF**: SolderWirePad_single_0-8mmDrill, Wire_Pads:SolderWirePad_single_0-8mmDrill, F.Cu at (123.1, 104.8)
- added REF**: SolderWirePad_single_0-8mmDrill, Wire_Pads:SolderWirePad_single_0-8mmDrill, F.Cu at (130.7, 104.8)
- added REF**: SolderWirePad_single_0-8mmDrill, Wire_Pads:SolderWirePad_single_0-8mmDrill, F.Cu at (128.2, 99.8)
- added REF**: SolderWirePad_single_0-8mmDrill, Wire_Pads:SolderWirePad_single_0-8mmDrill, F.Cu at (130.7, 99.8)
- added REF**: SolderWirePad_single_0-8mmDrill, Wire_Pads:SolderWirePad_single_0-8mmDrill, F.Cu at (125.6, 102.3)
- added REF**: SolderWirePad_single_0-8mmDrill, Wire_Pads:SolderWirePad_single_0-8mmDrill, F.Cu at (128.2, 104.8)
- added REF**: SolderWirePad_single_0-8mmDrill, Wire_Pads:SolderWirePad_single_0-8mmDrill, F.Cu at (123.1, 102.3)
- added REF**: SolderWirePad_single_0-8mmDrill, Wire_Pads:SolderWirePad_single_0-8mmDrill, F.Cu at (130.7, 102.3)
- added REF**: SolderWirePad_single_0-8mmDrill, Wire_Pads:SolderWirePad_single_0-8mmDrill, F.Cu at (128.2, 102.3)
- added REF**: SolderWirePad_single_0-8mmDrill, Wire_Pads:SolderWirePad_single_0-8mmDrill, F.Cu at (125.6, 99.8)
- added REF**: SolderWirePad_single_0-8mmDrill, Wire_Pads:SolderWirePad_single_0-8mmDrill, F.Cu at (138.4, 102.3)
- added REF**: SolderWirePad_single_0-8mmDrill, Wire_Pads:SolderWirePad_single_0-8mmDrill, F.Cu at (123.1, 99.8)
- added REF**: SolderWirePad_single_0-8mmDrill, Wire_Pads:SolderWirePad_single_0-8mmDrill, F.Cu at (120.5, 135.3)
- added REF**: SolderWirePad_single_0-8mmDrill, Wire_Pads:SolderWirePad_single_0-8mmDrill, F.Cu at (117.9, 135.3)
- added REF**: SolderWirePad_single_0-8mmDrill, Wire_Pads:SolderWirePad_single_0-8mmDrill, F.Cu at (115.4, 135.3)
- added REF**: SolderWirePad_single_0-8mmDrill, Wire_Pads:SolderWirePad_single_0-8mmDrill, F.Cu at (112.8, 135.3)
- added REF**: SolderWirePad_single_0-8mmDrill, Wire_Pads:SolderWirePad_single_0-8mmDrill, F.Cu at (110.3, 135.3)
- added REF**: SolderWirePad_single_0-8mmDrill, Wire_Pads:SolderWirePad_single_0-8mmDrill, F.Cu at (107.8, 135.3)
- added REF**: SolderWirePad_single_0-8mmDrill, Wire_Pads:SolderWirePad_single_0-8mmDrill, F.Cu at (120.5, 132.8)
- added REF**: SolderWirePad_single_0-8mmDrill, Wire_Pads:SolderWirePad_single_0-8mmDrill, F.Cu at (117.9, 132.8)
- added REF**: SolderWirePad_single_0-8mmDrill, Wire_Pads:SolderWirePad_single_0-8mmDrill, F.Cu at (115.4, 132.8)
- added REF**: SolderWirePad_single_0-8mmDrill, Wire_Pads:SolderWirePad_single_0-8mmDrill, F.Cu at (135.9, 99.8)
- added REF**: SolderWirePad_single_0-8mmDrill, Wire_Pads:SolderWirePad_single_0-8mmDrill, F.Cu at (112.8, 132.8)
- added REF**: SolderWirePad_single_0-8mmDrill, Wire_Pads:SolderWirePad_single_0-8mmDrill, F.Cu at (110.3, 132.8)
- added REF**: SolderWirePad_single_0-8mmDrill, Wire_Pads:SolderWirePad_single_0-8mmDrill, F.Cu at (107.8, 132.8)
- added REF**: SolderWirePad_single_0-8mmDrill, Wire_Pads:SolderWirePad_single_0-8mmDrill, F.Cu at (120.5, 130.2)
- added REF**: SolderWirePad_single_0-8mmDrill, Wire_Pads:SolderWirePad_single_0-8mmDrill, F.Cu at (117.9, 130.2)
- added REF**: SolderWirePad_single_0-8mmDrill, Wire_Pads:SolderWirePad_single_0-8mmDrill, F.Cu at (115.4, 130.2)
- added REF**: SolderWirePad_single_0-8mmDrill, Wire_Pads:SolderWirePad_single_0-8mmDrill, F.Cu at (112.8, 130.2)
- added REF**: SolderWirePad_single_0-8mmDrill, Wire_Pads:SolderWirePad_single_0-8mmDrill, F.Cu at (110.3, 130.2)
- added REF**: SolderWirePad_single_0-8mmDrill, Wire_Pads:SolderWirePad_single_0-8mmDrill, F.Cu at (107.8, 130.2)
- added REF**: SolderWirePad_single_0-8mmDrill, Wire_Pads:SolderWirePad_single_0-8mmDrill, F.Cu at (120.5, 127.7)
- added REF**: SolderWirePad_single_0-8mmDrill, Wire_Pads:SolderWirePad_single_0-8mmDrill, F.Cu at (140.9, 102.3)
- added REF**: SolderWirePad_single_0-8mmDrill, Wire_Pads:SolderWirePad_single_0-8mmDrill, F.Cu at (117.9, 127.7)
- added REF**: SolderWirePad_single_0-8mmDrill, Wire_Pads:SolderWirePad_single_0-8mmDrill, F.Cu at (115.4, 127.7)
- added REF**: SolderWirePad_single_0-8mmDrill, Wire_Pads:SolderWirePad_single_0-8mmDrill, F.Cu at (112.8, 127.7)
- added REF**: SolderWirePad_single_0-8mmDrill, Wire_Pads:SolderWirePad_single_0-8mmDrill, F.Cu at (110.3, 127.7)
- added REF**: SolderWirePad_single_0-8mmDrill, Wire_Pads:SolderWirePad_single_0-8mmDrill, F.Cu at (107.8, 127.7)
- added REF**: SolderWirePad_single_0-8mmDrill, Wire_Pads:SolderWirePad_single_0-8mmDrill, F.Cu at (120.5, 125.2)
- added REF**: SolderWirePad_single_0-8mmDrill, Wire_Pads:SolderWirePad_single_0-8mmDrill, F.Cu at (117.9, 125.2)
- added REF**: SolderWirePad_single_0-8mmDrill, Wire_Pads:SolderWirePad_single_0-8mmDrill, F.Cu at (115.4, 125.2)
- added REF**: SolderWirePad_single_0-8mmDrill, Wire_Pads:SolderWirePad_single_0-8mmDrill, F.Cu at (112.8, 125.2)
- added REF**: SolderWirePad_single_0-8mmDrill, Wire_Pads:SolderWirePad_single_0-8mmDrill, F.Cu at (110.3, 125.2)
- added REF**: SolderWirePad_single_0-8mmDrill, Wire_Pads:SolderWirePad_single_0-8mmDrill, F.Cu at (133.3, 99.8)
- added REF**: SolderWirePad_single_0-8mmDrill, Wire_Pads:SolderWirePad_single_0-8mmDrill, F.Cu at (107.8, 125.2)
- added REF**: SolderWirePad_single_0-8mmDrill, Wire_Pads:SolderWirePad_single_0-8mmDrill, F.Cu at (120.5, 122.6)
- added REF**: SolderWirePad_single_0-8mmDrill, Wire_Pads:SolderWirePad_single_0-8mmDrill, F.Cu at (117.9, 122.6)
- added REF**: SolderWirePad_single_0-8mmDrill, Wire_Pads:SolderWirePad_single_0-8mmDrill, F.Cu at (115.4, 122.6)
- added REF**: SolderWirePad_single_0-8mmDrill, Wire_Pads:SolderWirePad_single_0-8mmDrill, F.Cu at (112.8, 122.6)
- added REF**: SolderWirePad_single_0-8mmDrill, Wire_Pads:SolderWirePad_single_0-8mmDrill, F.Cu at (110.3, 122.6)
- added REF**: SolderWirePad_single_0-8mmDrill, Wire_Pads:SolderWirePad_single_0-8mmDrill, F.Cu at (107.8, 122.6)
- added REF**: SolderWirePad_single_0-8mmDrill, Wire_Pads:SolderWirePad_single_0-8mmDrill, F.Cu at (120.5, 120.1)
- added REF**: SolderWirePad_single_0-8mmDrill, Wire_Pads:SolderWirePad_single_0-8mmDrill, F.Cu at (117.9, 120.1)
- added REF**: SolderWirePad_single_0-8mmDrill, Wire_Pads:SolderWirePad_single_0-8mmDrill, F.Cu at (115.4, 120.1)
- added REF**: SolderWirePad_single_0-8mmDrill, Wire_Pads:SolderWirePad_single_0-8mmDrill, F.Cu at (135.9, 102.3)
- added REF**: SolderWirePad_single_0-8mmDrill, Wire_Pads:SolderWirePad_single_0-8mmDrill, F.Cu at (112.8, 120.1)
- added REF**: SolderWirePad_single_0-8mmDrill, Wire_Pads:SolderWirePad_single_0-8mmDrill, F.Cu at (110.3, 120.1)
- added REF**: SolderWirePad_single_0-8mmDrill, Wire_Pads:SolderWirePad_single_0-8mmDrill, F.Cu at (107.8, 120.1)
- added REF**: SolderWirePad_single_0-8mmDrill, Wire_Pads:SolderWirePad_single_0-8mmDrill, F.Cu at (120.5, 117.5)
- added REF**: SolderWirePad_single_0-8mmDrill, Wire_Pads:SolderWirePad_single_0-8mmDrill, F.Cu at (117.9, 117.5)
- added REF**: SolderWirePad_single_0-8mmDrill, Wire_Pads:SolderWirePad_single_0-8mmDrill, F.Cu at (115.4, 117.5)
- added REF**: SolderWirePad_single_0-8mmDrill, Wire_Pads:SolderWirePad_single_0-8mmDrill, F.Cu at (112.8, 117.5)
- added REF**: SolderWirePad_single_0-8mmDrill, Wire_Pads:SolderWirePad_single_0-8mmDrill, F.Cu at (110.3, 117.5)
- added REF**: SolderWirePad_single_0-8mmDrill, Wire_Pads:SolderWirePad_single_0-8mmDrill, F.Cu at (107.8, 117.5)
- added REF**: SolderWirePad_single_0-8mmDrill, Wire_Pads:SolderWirePad_single_0-8mmDrill, F.Cu at (120.5, 115.0)
- added REF**: SolderWirePad_single_0-8mmDrill, Wire_Pads:SolderWirePad_single_0-8mmDrill, F.Cu at (123.1, 110.0)
- added REF**: SolderWirePad_single_0-8mmDrill, Wire_Pads:SolderWirePad_single_0-8mmDrill, F.Cu at (117.9, 115.0)
- added REF**: SolderWirePad_single_0-8mmDrill, Wire_Pads:SolderWirePad_single_0-8mmDrill, F.Cu at (115.4, 115.0)
- added REF**: SolderWirePad_single_0-8mmDrill, Wire_Pads:SolderWirePad_single_0-8mmDrill, F.Cu at (112.8, 115.0)
- added REF**: SolderWirePad_single_0-8mmDrill, Wire_Pads:SolderWirePad_single_0-8mmDrill, F.Cu at (110.3, 115.0)
- added REF**: SolderWirePad_single_0-8mmDrill, Wire_Pads:SolderWirePad_single_0-8mmDrill, F.Cu at (107.8, 115.0)
- added REF**: SolderWirePad_single_0-8mmDrill, Wire_Pads:SolderWirePad_single_0-8mmDrill, F.Cu at (120.5, 112.5)
- added REF**: SolderWirePad_single_0-8mmDrill, Wire_Pads:SolderWirePad_single_0-8mmDrill, F.Cu at (117.9, 112.5)
- added REF**: SolderWirePad_single_0-8mmDrill, Wire_Pads:SolderWirePad_single_0-8mmDrill, F.Cu at (115.4, 112.5)
- added REF**: SolderWirePad_single_0-8mmDrill, Wire_Pads:SolderWirePad_single_0-8mmDrill, F.Cu at (112.8, 112.5)
- added REF**: SolderWirePad_single_0-8mmDrill, Wire_Pads:SolderWirePad_single_0-8mmDrill, F.Cu at (110.3, 112.5)
- added REF***: KiCad-Logo2_6mm_SilkScreen, Symbols:KiCad-Logo2_6mm_SilkScreen, B.Cu at (140.8, 119.2)
- added V14_19: AUTO_VIA, VIA_MATRIX, F.Cu at (130.1, 138.9)
- added V14_21: AUTO_VIA, VIA_MATRIX, F.Cu at (130.1, 144.0)
- added V15_16: AUTO_VIA, VIA_MATRIX, F.Cu at (132.7, 131.3)
- added V15_17: AUTO_VIA, VIA_MATRIX, F.Cu at (132.7, 133.8)
- added V15_18: AUTO_VIA, VIA_MATRIX, F.Cu at (132.7, 136.4)
- added V15_20: AUTO_VIA, VIA_MATRIX, F.Cu at (132.7, 141.4)
- added V15_7: AUTO_VIA, VIA_MATRIX, F.Cu at (132.7, 108.4)
- added V16_19: AUTO_VIA, VIA_MATRIX, F.Cu at (135.2, 138.9)
- added V17_20: AUTO_VIA, VIA_MATRIX, F.Cu at (137.7, 141.4)
- added V18_18: AUTO_VIA, VIA_MATRIX, F.Cu at (140.3, 136.4)
- added V19_18: AUTO_VIA, VIA_MATRIX, F.Cu at (142.8, 136.4)
- added V19_3: AUTO_VIA, VIA_MATRIX, F.Cu at (142.8, 98.3)
- added V19_4: AUTO_VIA, VIA_MATRIX, F.Cu at (142.8, 100.8)
- added V20_18: AUTO_VIA, VIA_MATRIX, F.Cu at (145.4, 136.4)
- added V21_18: AUTO_VIA, VIA_MATRIX, F.Cu at (147.9, 136.4)
- added V21_3: AUTO_VIA, VIA_MATRIX, F.Cu at (147.9, 98.3)
- added V22_18: AUTO_VIA, VIA_MATRIX, F.Cu at (150.4, 136.4)
- added V23_18: AUTO_VIA, VIA_MATRIX, F.Cu at (153.0, 136.4)
- added V23_21: AUTO_VIA, VIA_MATRIX, F.Cu at (153.0, 144.0)
- added V24_18: AUTO_VIA, VIA_MATRIX, F.Cu at (155.5, 136.4)
- added V25_18: AUTO_VIA, VIA_MATRIX, F.Cu at (158.1, 136.4)
- added V26_18: AUTO_VIA, VIA_MATRIX, F.Cu at (160.6, 136.4)
- added V27_18: AUTO_VIA, VIA_MATRIX, F.Cu at (163.1, 136.4)
- added V28_18: AUTO_VIA, VIA_MATRIX, F.Cu at (165.7, 136.4)
- added V28_19: AUTO_VIA, VIA_MATRIX, F.Cu at (165.7, 138.9)
- added V29_18: AUTO_VIA, VIA_MATRIX, F.Cu at (168.2, 136.4)
- added V29_19: AUTO_VIA, VIA_MATRIX, F.Cu at (168.2, 138.9)
- added V29_20: AUTO_VIA, VIA_MATRIX, F.Cu at (168.2, 141.4)
- added V29_5: AUTO_VIA, VIA_MATRIX, F.Cu at (168.2, 103.3)
- added V30_18: AUTO_VIA, VIA_MATRIX, F.Cu at (170.8, 136.4)
- added V30_2: AUTO_VIA, VIA_MATRIX, F.Cu at (170.8, 95.7)
- added V30_20: AUTO_VIA, VIA_MATRIX, F.Cu at (170.8, 141.4)
- added V30_21: AUTO_VIA, VIA_MATRIX, F.Cu at (170.8, 144.0)
- added V30_3: AUTO_VIA, VIA_MATRIX, F.Cu at (170.8, 98.3)
- added V30_4: AUTO_VIA, VIA_MATRIX, F.Cu at (170.8, 100.8)
- added V30_5: AUTO_VIA, VIA_MATRIX, F.Cu at (170.8, 103.3)
- added V6_2: AUTO_VIA, VIA_MATRIX, F.Cu at (109.8, 95.7)
- added V6_3: AUTO_VIA, VIA_MATRIX, F.Cu at (109.8, 98.3)
- added V7_2: AUTO_VIA, VIA_MATRIX, F.Cu at (112.3, 95.7)
- added V8_2: AUTO_VIA, VIA_MATRIX, F.Cu at (114.9, 95.7)
- added V9_2: AUTO_VIA, VIA_MATRIX, F.Cu at (117.4, 95.7)
- REF**: moved to B.Cu
- moved REF** 44.4 mm to (155.0, 120.2), turned to 180 degrees
- moved SW1 40.6 mm to (107.2, 139.8), turned to 0 degrees
- moved V12_19 3.57 mm to (125.0, 138.9)
- moved V12_20 3.57 mm to (125.0, 141.4)
- moved V12_21 3.57 mm to (125.0, 144.0)
- moved V12_3 3.57 mm to (125.0, 98.3)
- moved V10_19 3.57 mm to (120.0, 138.9)
- moved V10_20 3.57 mm to (120.0, 141.4)
- moved V10_3 3.57 mm to (120.0, 98.3)
- moved V11_19 3.57 mm to (122.5, 138.9)
- moved V11_20 3.57 mm to (122.5, 141.4)
- moved V11_21 3.57 mm to (122.5, 144.0)
- moved V11_3 3.57 mm to (122.5, 98.3)
- moved V13_19 3.57 mm to (127.6, 138.9)
- moved V13_20 3.57 mm to (127.6, 141.4)
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Connections:
- A1 pad 1: Net-(A1-Pad1) -> (no net)
- A1 pad 10: Net-(A1-Pad10) -> (no net)
- A1 pad 11: Net-(A1-Pad11) -> (no net)
- A1 pad 12: Net-(A1-Pad12) -> (no net)
- A1 pad 13: Net-(A1-Pad13) -> (no net)
- A1 pad 14: Net-(A1-Pad14) -> (no net)
- A1 pad 2: Net-(A1-Pad2) -> (no net)
- A1 pad 24: Net-(A1-Pad24) -> (no net)
- A1 pad 25: Net-(A1-Pad25) -> (no net)
- A1 pad 26: Net-(A1-Pad26) -> (no net)
- A1 pad 27: Net-(A1-Pad27) -> (no net)
- A1 pad 28: Net-(A1-Pad28) -> (no net)
- A1 pad 30: Net-(A1-Pad30) -> (no net)
- A1 pad 31: Net-(A1-Pad31) -> (no net)
- A1 pad 32: Net-(A1-Pad32) -> (no net)
- A1 pad 4: Net-(A1-Pad4) -> (no net)
- A1 pad 8: Net-(A1-Pad8) -> (no net)
- A1 pad 9: Net-(A1-Pad9) -> (no net)
Routing:
- net Net-(A1-Pad3): track 60.5 -> 32.5 mm
Other:
- board text added: "COM"
- board text added: "P1"
- board text added: "P2"
- board text added: "REV. 0.2"
- board text added: "Relay Shield"
- board text removed: "30A Relay Shield"
- board text removed: "REV. 0.1"
