File: mysensors/node/pro_mini/pro_mini.kicad_pcb (KiCad board)
At the start: 2 copper layers, 50.5 x 29.9 mm, 141 parts, among them IC1 ArduinoProMini, U1 NRF24L01, U2 NCP1402

Commit message: mys pro mini refactorings
Parts:
- removed the REF** at (147.5, 115.5)
- removed V10_10 (x5), V10_3 (x3), V11_10, V12_10, V14_10, V15_4, V15_5, V17_5, V18_10 (x4), V19_5, V19_7, V19_8, V20_5, V20_6, V20_7, V20_8, V21_5, V21_7, V21_8, V22_5, V22_6, V22_7, V22_8, V23_5, V23_6, V23_7, V23_8 (x2), V24_5, V24_6, V24_7, V24_8 (x2), V25_4, V25_8, V26_4, V27_4, V28_4, V28_5, V28_6 (x2), V29_5, V29_6, V29_7, V30_6, V30_7, V31_6, V33_8, V34_7, V35_6, V36_9 (x9), V37_9 (x2), V38_9: AUTO_VIA, VIA_MATRIX
- added U1: NRF24L01, mysensors_radios:NRF24L01, F.Cu at (144.3, 90.0)
- added V10_8: AUTO_VIA, VIA_MATRIX, F.Cu at (117.6, 104.8)
- added V11_4: AUTO_VIA, VIA_MATRIX, F.Cu at (119.6, 96.8)
- added V11_8: AUTO_VIA, VIA_MATRIX, F.Cu at (119.6, 104.8)
- added V12_8: AUTO_VIA, VIA_MATRIX, F.Cu at (121.6, 104.8)
- added V13_8: AUTO_VIA, VIA_MATRIX, F.Cu at (123.6, 104.8)
- added V16_4: AUTO_VIA, VIA_MATRIX, F.Cu at (129.6, 96.8)
- added V16_5: AUTO_VIA, VIA_MATRIX, F.Cu at (129.6, 98.8)
- added V16_6: AUTO_VIA, VIA_MATRIX, F.Cu at (129.6, 100.8)
- added V18_3: AUTO_VIA, VIA_MATRIX, F.Cu at (133.6, 94.8)
- added V18_4: AUTO_VIA, VIA_MATRIX, F.Cu at (133.6, 96.8)
- added V18_6: AUTO_VIA, VIA_MATRIX, F.Cu at (145.4, 101.6)
- added V18_6: AUTO_VIA, VIA_MATRIX, F.Cu at (159.5, 99.2)
- added V18_6: AUTO_VIA, VIA_MATRIX, F.Cu at (159.4, 101.5)
- added V18_6: AUTO_VIA, VIA_MATRIX, F.Cu at (159.5, 97.1)
- added V18_6: AUTO_VIA, VIA_MATRIX, F.Cu at (148.0, 101.7)
- added V18_6: AUTO_VIA, VIA_MATRIX, F.Cu at (151.0, 99.0)
- added V18_6: AUTO_VIA, VIA_MATRIX, F.Cu at (152.1, 101.8)
- added V18_6: AUTO_VIA, VIA_MATRIX, F.Cu at (133.6, 100.8)
- added V21_4: AUTO_VIA, VIA_MATRIX, F.Cu at (139.6, 96.8)
- added V7_1: AUTO_VIA, VIA_MATRIX, F.Cu at (111.6, 90.8)
- added V7_2: AUTO_VIA, VIA_MATRIX, F.Cu at (111.6, 92.8)
- added V7_5: AUTO_VIA, VIA_MATRIX, F.Cu at (111.3, 98.8)
- added V7_6: AUTO_VIA, VIA_MATRIX, F.Cu at (111.3, 100.8)
- added V7_7: AUTO_VIA, VIA_MATRIX, F.Cu at (111.3, 102.8)
- added V9_8: AUTO_VIA, VIA_MATRIX, F.Cu at (115.6, 104.8)
- moved V21_6 10.9 mm to (139.6, 100.8)
- moved V19_6 9.91 mm to (135.6, 100.8)
- moved V18_5 9.30 mm to (133.6, 98.8)
- moved R2 4.65 mm to (130.1, 94.3)
- moved R1 3.88 mm to (131.8, 98.3), turned to 90 degrees
Connections:
- REF** pad : (no net) -> GND (x4)
- REF** pad : (no net) -> +3.3V (x4)
- REF** pad : (no net) -> Net-(IC1-Pad11)
- REF** pad : (no net) -> Net-(IC1-Pad10)
- REF** pad : (no net) -> Net-(IC1-Pad9)
- REF** pad : (no net) -> Net-(IC1-Pad8)
- REF** pad : (no net) -> Net-(IC1-Pad7)
Routing:
- net +3.3V: track 58.8 -> 100.6 mm, vias 1 -> 2
- net (no net): track 0.00 -> 34.7 mm
- net /RF_SCK: track 21.1 -> 36.0 mm, vias 0 -> 1
- net /RF_MOSI: track 17.2 -> 31.3 mm
- net /RF_MISO: track 16.0 -> 28.3 mm
- net GND: track 15.5 -> 25.4 mm, vias 0 -> 1
- net Net-(BT1-Pad1): track 18.6 -> 24.0 mm
- net /RF_CE: track 23.8 -> 28.4 mm
- net /RF_IRQ: track 32.8 -> 36.6 mm, vias 0 -> 2
- net Net-(IC1-Pad9): track 0.00 -> 3.30 mm
- net Net-(IC1-Pad8): track 0.00 -> 3.30 mm
- net Net-(IC1-Pad7): track 0.00 -> 3.30 mm
- net Net-(IC1-Pad11): track 0.00 -> 3.30 mm
- net Net-(IC1-Pad10): track 0.00 -> 3.30 mm
- net /RF_CSN: track 20.6 -> 18.6 mm
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Other:
- board size 50.5 x 29.9 mm -> 50.5 x 30.1 mm
- board text added: "REV. 0.2"
- board text removed: "REV. 0.1"
