File: other/rpi_zero_ws2812/rpi_zero_ws2812.kicad_pcb (KiCad board)
At the start: 2 copper layers, 65 x 30 mm, 36 parts, among them J1 RPI_Zero, J2 5V INPUT, J4 WS2812, Q1 BSS138, U2 AMS1117, U3 DS18B20

Commit message: rpi zero ws2812 final touches
Parts:
- added REF**: 1pin, myfootprints:1pin, F.Cu at (155.9, 95.3)
- added REF**: 1pin, myfootprints:1pin, F.Cu at (149.9, 95.3)
- added REF**: 1pin, myfootprints:1pin, F.Cu at (151.9, 95.3)
- added REF**: 1pin, myfootprints:1pin, F.Cu at (153.9, 95.3)
- moved R2 0.25 mm to (157.9, 94.5)
Connections:
- REF** pad : (no net) -> +3V3 (x4)
Routing:
- net (no net): track 0.00 -> 22.5 mm
- net +3V3: track 39.9 -> 42.2 mm, vias 1 -> 2
