File: other/Bicycle_Lights/kicad/BL_PCB_latest.kicad_pcb (KiCad board)
At the start: 2 copper layers, 136.9 x 67.1 mm, 159 parts, among them J2 SWD, Q1 MMBT2222, Q2 MMBT2222, Q3 MMBT2222, Q4 MMBT2222, Q5 MMBT2222, Q6 MMBT2222, U1 E73-2G4M0S

Commit message: bl prj update
Routing:
- net Q2_3: track 101.0 -> 99.0 mm
