File: IOT/node/livolo_EU_switch/VL-C700X-1_Ver_C2/Power_Supply/kicad/NRF52832_Touch_Switch_Power_Supply.kicad_pcb (KiCad board)
At the start: 2 copper layers, 46 x 43.4 mm, 56 parts, among them CN1 2X7P, K1 HFE60-12-1HT-L2, K2 HFE60-12-1HT-L2, Q1 IRLR8726PBF, Q2 MMBT3904, T1 EE10A-1, U1 LM321, U2 MCP1703T-3302, U3 EL357, U4 LNK364DN-TL, U6 TPL7407LPWR

Commit message: ref
Changed lines of the file:
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@@
     (last_trace_width 0.25)
     (trace_clearance 0.2)
-    (zone_clearance 0.5)
+    (zone_clearance 1)
     (zone_45_only no)
     (trace_min 0.2)
@@
     (at 133.604 55.202 90)
     (attr smd)
-    (fp_text reference R19 (at -1.186 0.023 90) (layer B.SilkS)
+    (fp_text reference R19 (at -1.478 0.826 180) (layer B.SilkS)
       (effects (font (size 0.508 0.508) (thickness 0.076)) (justify left mirror))
     )
@@
   )
   (zone (net 13) (net_name GND) (layer F.Cu) (hatch edge 0.508)
-    (connect_pads yes (clearance 0.5))
-    (min_thickness 0.5)
+    (connect_pads yes (clearance 1))
+    (min_thickness 0.125)
     (fill yes (arc_segments 32) (thermal_gap 0.508) (thermal_bridge_width 0.508) (smoothing fillet))
     (polygon
       (pts
-        (xy 137.905752 58.760771) (xy 137.795 61.015165) (xy 137.463813 63.247848) (xy 136.915379 65.437318) (xy 136.154981 67.562489)
-        (xy 135.189941 69.602895) (xy 134.029553 71.538886) (xy 132.684992 73.351816) (xy 131.169207 75.024226) (xy 129.496797 76.540011)
-        (xy 127.683867 77.884572) (xy 125.747876 79.04496) (xy 123.70747 80.01) (xy 121.582299 80.770398) (xy 119.392829 81.318832)
-        (xy 117.160146 81.650019) (xy 114.905752 81.760771) (xy 112.651358 81.650019) (xy 110.418675 81.318832) (xy 108.229205 80.770398)
-        (xy 106.104034 80.01) (xy 104.063628 79.04496) (xy 102.127637 77.884572) (xy 100.314707 76.540011) (xy 98.642297 75.024226)
-        (xy 97.126512 73.351816) (xy 95.781951 71.538886) (xy 94.621563 69.602895) (xy 93.656523 67.562489) (xy 92.896125 65.437318)
-        (xy 92.347691 63.247848) (xy 92.016504 61.015165) (xy 91.905752 58.760771) (xy 92.016504 56.506377) (xy 92.347691 54.273694)
-        (xy 92.896125 52.084224) (xy 93.656523 49.959053) (xy 94.621563 47.918647) (xy 95.781951 45.982656) (xy 97.126512 44.169726)
-        (xy 98.642297 42.497316) (xy 100.314707 40.981531) (xy 102.127637 39.63697) (xy 104.063628 38.476582) (xy 106.104034 37.511542)
-        (xy 108.229205 36.751144) (xy 110.418675 36.20271) (xy 112.651358 35.871523) (xy 114.905752 35.760771) (xy 117.160146 35.871523)
-        (xy 119.392829 36.20271) (xy 121.582299 36.751144) (xy 123.70747 37.511542) (xy 125.747876 38.476582) (xy 127.683867 39.63697)
-        (xy 129.496797 40.981531) (xy 131.169207 42.497316) (xy 132.684992 44.169726) (xy 134.029553 45.982656) (xy 135.189941 47.918647)
-        (xy 136.154981 49.959053) (xy 136.915379 52.084224) (xy 137.463813 54.273694) (xy 137.795 56.506377)
+        (xy 137.834396 58.47157) (xy 137.723644 60.725964) (xy 137.392457 62.958647) (xy 136.844023 65.148117) (xy 136.083625 67.273288)
+        (xy 135.118585 69.313694) (xy 133.958197 71.249685) (xy 132.613636 73.062615) (xy 131.097851 74.735025) (xy 129.425441 76.25081)
+        (xy 127.612511 77.595371) (xy 125.67652 78.755759) (xy 123.636114 79.720799) (xy 121.510943 80.481197) (xy 119.321473 81.029631)
+        (xy 117.08879 81.360818) (xy 114.834396 81.47157) (xy 112.580002 81.360818) (xy 110.347319 81.029631) (xy 108.157849 80.481197)
+        (xy 106.032678 79.720799) (xy 103.992272 78.755759) (xy 102.056281 77.595371) (xy 100.243351 76.25081) (xy 98.570941 74.735025)
+        (xy 97.055156 73.062615) (xy 95.710595 71.249685) (xy 94.550207 69.313694) (xy 93.585167 67.273288) (xy 92.824769 65.148117)
+        (xy 92.276335 62.958647) (xy 91.945148 60.725964) (xy 91.834396 58.47157) (xy 91.945148 56.217176) (xy 92.276335 53.984493)
+        (xy 92.824769 51.795023) (xy 93.585167 49.669852) (xy 94.550207 47.629446) (xy 95.710595 45.693455) (xy 97.055156 43.880525)
+        (xy 98.570941 42.208115) (xy 100.243351 40.69233) (xy 102.056281 39.347769) (xy 103.992272 38.187381) (xy 106.032678 37.222341)
+        (xy 108.157849 36.461943) (xy 110.347319 35.913509) (xy 112.580002 35.582322) (xy 114.834396 35.47157) (xy 117.08879 35.582322)
+        (xy 119.321473 35.913509) (xy 121.510943 36.461943) (xy 123.636114 37.222341) (xy 125.67652 38.187381) (xy 127.612511 39.347769)
+        (xy 129.425441 40.69233) (xy 131.097851 42.208115) (xy 132.613636 43.880525) (xy 133.958197 45.693455) (xy 135.118585 47.629446)
+        (xy 136.083625 49.669852) (xy 136.844023 51.795023) (xy 137.392457 53.984493) (xy 137.723644 56.217176)
       )
     )
   )
   (zone (net 13) (net_name GND) (layer B.Cu) (hatch edge 0.508)
-    (connect_pads yes (clearance 0.5))
-    (min_thickness 0.5)
+    (connect_pads yes (clearance 1))
+    (min_thickness 0.125)
     (fill yes (arc_segments 32) (thermal_gap 0.508) (thermal_bridge_width 0.508) (smoothing fillet))
     (polygon
       (pts
-        (xy 137.905752 58.760771) (xy 137.795 61.015165) (xy 137.463813 63.247848) (xy 136.915379 65.437318) (xy 136.154981 67.562489)
-        (xy 135.189941 69.602895) (xy 134.029553 71.538886) (xy 132.684992 73.351816) (xy 131.169207 75.024226) (xy 129.496797 76.540011)
-        (xy 127.683867 77.884572) (xy 125.747876 79.04496) (xy 123.70747 80.01) (xy 121.582299 80.770398) (xy 119.392829 81.318832)
-        (xy 117.160146 81.650019) (xy 114.905752 81.760771) (xy 112.651358 81.650019) (xy 110.418675 81.318832) (xy 108.229205 80.770398)
-        (xy 106.104034 80.01) (xy 104.063628 79.04496) (xy 102.127637 77.884572) (xy 100.314707 76.540011) (xy 98.642297 75.024226)
-        (xy 97.126512 73.351816) (xy 95.781951 71.538886) (xy 94.621563 69.602895) (xy 93.656523 67.562489) (xy 92.896125 65.437318)
-        (xy 92.347691 63.247848) (xy 92.016504 61.015165) (xy 91.905752 58.760771) (xy 92.016504 56.506377) (xy 92.347691 54.273694)
-        (xy 92.896125 52.084224) (xy 93.656523 49.959053) (xy 94.621563 47.918647) (xy 95.781951 45.982656) (xy 97.126512 44.169726)
-        (xy 98.642297 42.497316) (xy 100.314707 40.981531) (xy 102.127637 39.63697) (xy 104.063628 38.476582) (xy 106.104034 37.511542)
-        (xy 108.229205 36.751144) (xy 110.418675 36.20271) (xy 112.651358 35.871523) (xy 114.905752 35.760771) (xy 117.160146 35.871523)
-        (xy 119.392829 36.20271) (xy 121.582299 36.751144) (xy 123.70747 37.511542) (xy 125.747876 38.476582) (xy 127.683867 39.63697)
-        (xy 129.496797 40.981531) (xy 131.169207 42.497316) (xy 132.684992 44.169726) (xy 134.029553 45.982656) (xy 135.189941 47.918647)
-        (xy 136.154981 49.959053) (xy 136.915379 52.084224) (xy 137.463813 54.273694) (xy 137.795 56.506377)
+        (xy 137.83 58.47) (xy 137.719248 60.724394) (xy 137.388061 62.957077) (xy 136.839627 65.146547) (xy 136.079229 67.271718)
+        (xy 135.114189 69.312124) (xy 133.953801 71.248115) (xy 132.60924 73.061045) (xy 131.093455 74.733455) (xy 129.421045 76.24924)
+        (xy 127.608115 77.593801) (xy 125.672124 78.754189) (xy 123.631718 79.719229) (xy 121.506547 80.479627) (xy 119.317077 81.028061)
+        (xy 117.084394 81.359248) (xy 114.83 81.47) (xy 112.575606 81.359248) (xy 110.342923 81.028061) (xy 108.153453 80.479627)
+        (xy 106.028282 79.719229) (xy 103.987876 78.754189) (xy 102.051885 77.593801) (xy 100.238955 76.24924) (xy 98.566545 74.733455)
+        (xy 97.05076 73.061045) (xy 95.706199 71.248115) (xy 94.545811 69.312124) (xy 93.580771 67.271718) (xy 92.820373 65.146547)
+        (xy 92.271939 62.957077) (xy 91.940752 60.724394) (xy 91.83 58.47) (xy 91.940752 56.215606) (xy 92.271939 53.982923)
+        (xy 92.820373 51.793453) (xy 93.580771 49.668282) (xy 94.545811 47.627876) (xy 95.706199 45.691885) (xy 97.05076 43.878955)
+        (xy 98.566545 42.206545) (xy 100.238955 40.69076) (xy 102.051885 39.346199) (xy 103.987876 38.185811) (xy 106.028282 37.220771)
+        (xy 108.153453 36.460373) (xy 110.342923 35.911939) (xy 112.575606 35.580752) (xy 114.83 35.47) (xy 117.084394 35.580752)
+        (xy 119.317077 35.911939) (xy 121.506547 36.460373) (xy 123.631718 37.220771) (xy 125.672124 38.185811) (xy 127.608115 39.346199)
+        (xy 129.421045 40.69076) (xy 131.093455 42.206545) (xy 132.60924 43.878955) (xy 133.953801 45.691885) (xy 135.114189 47.627876)
+        (xy 136.079229 49.668282) (xy 136.839627 51.793453) (xy 137.388061 53.982923) (xy 137.719248 56.215606)
       )
     )

Commit message: ref
Parts:
- C3: footprint easyeda:0805 -> Capacitor_Tantalum_SMD:CP_EIA-3528-21_Kemet-B; moved to B.Cu
- moved C3 0.58 mm to (115.8, 78.5), turned to 0 degrees
Routing:
- net GND: vias 47 -> 46

Commit message: eu switch rev0.4 - the last one
Parts:
- removed REF** (x3): MountingHole_2mm, MountingHole:MountingHole_2mm
- added ?: , AutoGenerated:MountingHole_1.50mm, F.Cu at (120.8, 43.3)
- added ?: , AutoGenerated:MountingHole_1.50mm, F.Cu at (102.1, 43.2)
- added ?: , AutoGenerated:MountingHole_1.50mm, F.Cu at (110.0, 78.5)
- C3: value 22uF -> CAP-SMD_L3.5-W2.8-R-RD; footprint Capacitor_Tantalum_SMD:CP_EIA-3528-21_Kemet-B -> easyeda:CAP-SMD_L3.5-W2.8-R-RD; moved to F.Cu
- moved C3 0.94 mm to (114.9, 78.7), turned to 180 degrees
- moved C5 0.74 mm to (128.8, 72.9)
- moved D15 0.67 mm to (123.6, 59.8)
- moved D14 0.64 mm to (123.4, 63.8)
- moved R2 0.45 mm to (115.4, 67.9)
- moved C1 0.38 mm to (118.2, 71.0)
- moved C11 0.38 mm to (121.8, 75.8)
- moved D3 0.26 mm to (112.6, 69.5)
- moved R20 0.25 mm to (125.7, 44.3)
- moved R7 0.15 mm to (115.1, 70.0), turned to 270 degrees
- moved C2 0.13 mm to (99.4, 70.1)
- turned R3 to 270 degrees
Connections:
- C3 pad 1: GND -> +3V3
- C3 pad 2: +3V3 -> GND
- C7 pad 1: (no net) -> R16_2
- D13 pad 2: (no net) -> D13_2
- R16 pad 2: (no net) -> R16_2
- R20 pad 2: (no net) -> D13_2
Routing:
- net (no net): track 24.4 -> 0.00 mm, vias 2 -> 0
- net D13_2: track 0.00 -> 22.6 mm, vias 0 -> 2
- net D1_1: track 56.5 -> 45.8 mm, vias 26 -> 23
- net GND: track 36.7 -> 39.3 mm, vias 46 -> 42
- net AC_DC_N: track 30.5 -> 33.0 mm, vias 5 -> 4
- net R16_2: track 0.00 -> 2.03 mm
- net U4_5: track 25.7 -> 24.5 mm, vias 1 -> 2
- net +12V: track 51.7 -> 52.6 mm
- net R2_2: track 19.4 -> 20.0 mm
- net U4_4: track 6.35 -> 6.84 mm, vias 0 -> 1
Other:
- board size 46 x 43.4 mm -> 46.8 x 44.3 mm
- rule pad_to_mask_clearance: 0.051 -> 0
- board text added: "REV. 0.4"
- board text removed: "REV. 0.3"
